File: PCB/OptiLogic-16-Pro.kicad_pcb (KiCad board)
At the start: 8 copper layers, 230 x 145.3 mm, 342 parts, among them J1 SFP, J2 SFP, J3 SFP, J4 USB_C_Receptacle, J5 Conn_02x07_Odd_Even, J6 Conn_02x10_Odd_Even, J7 Conn_02x10_Odd_Even, J8 Conn_Coaxial, J9 Barrel_Jack, Q2 Q_PMOS_GSD, SW1 SW_Push, U1 MT41K256M16HA, U22 REF5025AD, U26 Opamp_Quad, U27 Opamp_Quad, U28 Opamp_Quad, U29 Opamp_Quad, U3 KSZ9031RNXCA, U30 TPS563200, U31 AP2112K-2.5, U32 TLV75512PDBV, U33 TPS51200DRC, U34 TPS563200, U36 TPS563200, U4 W25Q128JVS, U42 FT601Q, U5 TPS563200, U6 LMH7324, U7 LMH7324, U8 LMH7324, U9 LMH7324, Y1 ACO-xxxMHz, Y2 125MHz, Y3 Crystal, Y4 25.000 MHz

Commit message: Fixed missing connections
Routing:
- net GND: track 1337.5 -> 1411.9 mm, vias 162 -> 165
- net +3V3: track 698.0 -> 747.0 mm, vias 40 -> 41
- net FT_RESET_N: track 43.7 -> 75.0 mm, vias 1 -> 3
- net JTAG_TDI: track 42.4 -> 64.7 mm, vias 0 -> 2
- net DDR_RESET_N: track 12.5 -> 34.1 mm, vias 1 -> 2
- net FPGA_D02: track 53.9 -> 33.4 mm, vias 5 -> 4
- net Net-(U37A-INIT_B_0): track 0.00 -> 18.2 mm, vias 0 -> 2
- net DDR_CK_N: track 15.7 -> 26.9 mm
- net +1V8: track 237.0 -> 247.1 mm, vias 29 -> 30
- net USCITA_FPGA_0_P: track 147.2 -> 138.5 mm, vias 4 -> 5
- net +1V5: track 304.8 -> 312.9 mm, vias 26 -> 28
- net DDR_DQ0: track 26.8 -> 33.8 mm
- net DDR_RAS_N: track 17.2 -> 23.4 mm
- net DDR_DQ6: track 29.1 -> 24.9 mm, vias 2 -> 3
- net USCITA_FPGA_4_P: track 96.9 -> 93.0 mm
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